Commit message: help

File: spider_description/urdf/spider1.urdf (robot description, URDF)
Before this commit: robot spider_description, 19 links, 18 joints
Links:
- link base_link: mass 0.6 -> 0.61161
- link link_c1_lf: mass 0.02 -> 0.020733
- link link_c1_lm: mass 0.02 -> 0.0207333939617732
- link link_c1_lr: mass 0.02 -> 0.0207333939617732
- link link_c1_rf: mass 0.02 -> 0.0207333939617732
- link link_c1_rm: mass 0.02 -> 0.0207333939617732
- link link_c1_rr: mass 0.02 -> 0.0207333939617732
- link link_thigh_lf: mass 0.09 -> 0.095338
- link link_thigh_lm: mass 0.09 -> 0.095338126082866
- link link_thigh_lr: mass 0.09 -> 0.0953381260778558
- link link_thigh_rf: mass 0.09 -> 0.0953381260778559
- link link_thigh_rm: mass 0.09 -> 0.0953381260828659
- link link_thigh_rr: mass 0.09 -> 0.0953381260778557
- link link_tibia_lf: mass 0.03 -> 0.027469
- link link_tibia_lm: mass 0.03 -> 0.0274685503185618
- link link_tibia_lr: mass 0.03 -> 0.0274685501932786
- link link_tibia_rf: mass 0.03 -> 0.0274685501932794
- link link_tibia_rm: mass 0.03 -> 0.0274685503185618
- link link_tibia_rr: mass 0.03 -> 0.027468550193276
