Commit message: начала делать движение ноги

File: spider_description/urdf/spider.urdf (robot description, URDF)
Before this commit: robot Hexapod_urdf_v1, 19 links, 18 joints
Links:
- link base_link: geometry collision mesh filename=package://spider_description/meshes/base_link.STL; visual mesh filename=package://spider_description/meshes/base_link.STL
- link link_c1_lf: geometry collision mesh filename=package://spider_description/meshes/link_c1_lf.STL; visual mesh filename=package://spider_description/meshes/link_c1_lf.STL
- link link_c1_lm: geometry collision mesh filename=package://spider_description/meshes/link_c1_lm.STL; visual mesh filename=package://spider_description/meshes/link_c1_lm.STL
- link link_c1_lr: geometry collision mesh filename=package://spider_description/meshes/link_c1_lr.STL; visual mesh filename=package://spider_description/meshes/link_c1_lr.STL
- link link_c1_rf: geometry collision mesh filename=package://spider_description/meshes/link_c1_rf.STL; visual mesh filename=package://spider_description/meshes/link_c1_rf.STL
- link link_c1_rm: geometry collision mesh filename=package://spider_description/meshes/link_c1_rm.STL; visual mesh filename=package://spider_description/meshes/link_c1_rm.STL
- link link_c1_rr: geometry collision mesh filename=package://spider_description/meshes/link_c1_rr.STL; visual mesh filename=package://spider_description/meshes/link_c1_rr.STL
- link link_thigh_lf: geometry collision mesh filename=package://spider_description/meshes/link_thigh_lf.STL; visual mesh filename=package://spider_description/meshes/link_thigh_lf.STL
- link link_thigh_lm: geometry collision mesh filename=package://spider_description/meshes/link_thigh_lm.STL; visual mesh filename=package://spider_description/meshes/link_thigh_lm.STL
- link link_thigh_lr: geometry collision mesh filename=package://spider_description/meshes/link_thigh_lr.STL; visual mesh filename=package://spider_description/meshes/link_thigh_lr.STL
- link link_thigh_rf: geometry collision mesh filename=package://spider_description/meshes/link_thigh_rf.STL; visual mesh filename=package://spider_description/meshes/link_thigh_rf.STL
- link link_thigh_rm: geometry collision mesh filename=package://spider_description/meshes/link_thigh_rm.STL; visual mesh filename=package://spider_description/meshes/link_thigh_rm.STL
- link link_thigh_rr: geometry collision mesh filename=package://spider_description/meshes/link_thigh_rr.STL; visual mesh filename=package://spider_description/meshes/link_thigh_rr.STL
- link link_tibia_lf: geometry collision mesh filename=package://spider_description/meshes/link_tibia_lf.STL; visual mesh filename=package://spider_description/meshes/link_tibia_lf.STL
- link link_tibia_lm: geometry collision mesh filename=package://spider_description/meshes/link_tibia_lm.STL; visual mesh filename=package://spider_description/meshes/link_tibia_lm.STL
- link link_tibia_lr: geometry collision mesh filename=package://spider_description/meshes/link_tibia_lr.STL; visual mesh filename=package://spider_description/meshes/link_tibia_lr.STL
- link link_tibia_rf: geometry collision mesh filename=package://spider_description/meshes/link_tibia_rf.STL; visual mesh filename=package://spider_description/meshes/link_tibia_rf.STL
- link link_tibia_rm: geometry collision mesh filename=package://spider_description/meshes/link_tibia_rm.STL; visual mesh filename=package://spider_description/meshes/link_tibia_rm.STL
- link link_tibia_rr: geometry collision mesh filename=package://spider_description/meshes/link_tibia_rr.STL; visual mesh filename=package://spider_description/meshes/link_tibia_rr.STL

Commit message: commit 19.02 попытка выровнять походку 126262

File: spider_description/urdf/spider.urdf (robot description, URDF)
Before this commit: robot spider_description, 19 links, 18 joints
Links:
- added link base
Joints:
- added joint base_joint: type fixed, parent base, child base_link, origin xyz=0.0 0.0 -0.7 rpy=0.0 0.0 0.0
- joint j_tibia_lf: limit lower=-2.2689 upper=2.2689 effort=6.0 velocity=0.524 -> lower=-3.1416 upper=3.1416 effort=6.0 velocity=0.524

File: spider_description/urdf/spider.xacro (robot description, xacro)
@@ -24,5 +24,5 @@
             <origin xyz="0.0 0.0 0.0" rpy="0.0 0.0 0.0"/>
             <geometry>
-                <mesh filename="package://spider/meshes/base_link.STL" />
+                <mesh filename="package://spider_description/meshes/xacro/base_link.STL" />
             </geometry>
             <material name="">
@@ -33,5 +33,5 @@
             <origin xyz="0.0 0.0 0.0" rpy="0.0 0.0 0.0"/>
             <geometry>
-                <mesh filename="package://spider/meshes/base_link.STL" />
+                <mesh filename="package://spider_description/meshes/xacro/base_link.STL" />
             </geometry>
             <material name="">
@@ -40,10 +40,16 @@
         </collision>
         <inertial>
-            <origin xyz="0.0 0.0 0.0" rpy="0.0 0.0 0.0" />
-            <mass value="0.00001"/>
-            <inertia
-                ixx="1.0" ixy="0.0"  ixz="0.0"
-                iyy="1.0" iyz="0.0"
-                izz="1.0" />
+        <origin
+                xyz="-0.000530634264644336 -0.000146735871100936 0.002797336519253"
+                rpy="0 0 0" />
+              <mass
+                value="0.611606451626775" />
+              <inertia
+                ixx="0.00454780272495035"
+                ixy="-5.85469596986661E-07"
+                ixz="5.809136780602E-06"
+                iyy="0.00784053245943273"
+                iyz="1.609753583614E-06"
+                izz="0.0121391274208026" />
         </inertial>
     </link>
@@ -54,5 +60,5 @@
    <xacro:property name="joint_velocity" value="0.524"/>
     <!-- Leg macro -->
-    <xacro:macro name="leg" params="side position x y angle axis">
+    <xacro:macro name="leg" params="side position x y angle axis_femur axis_tibia">
         <!-- leg position -->
         <joint name="leg_center_joint_${side}${position}" type="fixed">
@@ -72,8 +78,8 @@
         </link>
 <!-- coxa -->
-       <joint name="coxa_joint_${side}${position}" type="revolute">
+       <joint name="j_c1_${side}${position}" type="revolute">
            <origin xyz="0.0 0.0 0.0" rpy="0.0 0.0 ${angle}"/>
            <parent link="leg_center_${side}${position}"/>
-           <child link="coxa_${side}${position}"/>
+           <child link="link_c1_${side}${position}"/>
            <axis xyz="0.0 0.0 1.0"/>
            <limit lower="${joint_lower_limit}" upper="${joint_upper_limit}" effort="${joint_effort}" velocity="${joint_velocity}"/>
@@ -81,5 +87,5 @@
        <transmission name="coxa_transmission_${side}${position}">
            <type>transmission_interface/SimpleTransmission</type>
-           <joint name="coxa_joint_${side}${position}">
+           <joint name="j_c1_${side}${position}">
                <hardwareInterface>EffortJointInterface</hardwareInterface>
            </joint>
@@ -89,9 +95,9 @@
            </actuator>
        </transmission>
-       <link name="coxa_${side}${position}">
+       <link name="link_c1_${side}${position}">
            <visual>
                <origin xyz="0.0 0.0 0.0" rpy="0.0 0.0 0.0"/>
                <geometry>
-                   <mesh filename="package://spider/meshes/coxa_link.STL"/>
+                   <mesh filename="package://spider_description/meshes/xacro/coxa_link.STL"/>
                </geometry>
                <material name="">
@@ -102,5 +108,5 @@
                <origin xyz="0.0 0.0 0.0" rpy="0.0 0.0 0.0" />
                <geometry>
-                   <mesh filename="package://spider/meshes/coxa_link.STL"/>
+                   <mesh filename="package://spider_description/meshes/xacro/coxa_link.STL"/>
                </geometry>
                <material name="">
@@ -109,23 +115,29 @@
            </collision>
            <inertial>
-               <origin xyz="0.0 0.0 0.0" rpy="0.0 0.0 0.0" />
-               <mass value="0.00001"/>
-               <inertia
-                   ixx="1.0" ixy="0.0"  ixz="0.0"
-                   iyy="1.0" iyz="0.0"
-                   izz="1.0" />
+           <origin
+                   xyz="0.0259999991636717 5.48568285269058E-07 -5.52350892489561E-07"
+                   rpy="0 0 0" />
+                 <mass
+                   value="0.0207333939617734" />
+                 <inertia
+                   ixx="7.12966880670217E-06"
+                   ixy="-4.04797875390301E-11"
+                   ixz="-4.20782143594676E-11"
+                   iyy="7.05736504437165E-06"
+                   iyz="-7.44539286286323E-15"
+                   izz="7.05736451070854E-06" />
            </inertial>
        </link>
 <!-- femur -->
-        <joint name="femur_joint_${side}${position}" type="revolute">
+        <joint name="j_thigh_${side}${position}" type="revolute">
             <origin xyz="${coxa_length} 0.0 0.0" rpy="-${pi/2} 0 0.0"/>
-            <parent link="coxa_${side}${position}"/>
-            <child link="femur_${side}${position}"/>
-            <axis xyz="0.0 0.0 ${axis}"/>
+            <parent link="link_c1_${side}${position}"/>
+            <child link="link_thigh_${side}${position}"/>
+            <axis xyz="0.0 0.0 ${axis_femur}"/>
             <limit lower="${joint_lower_limit}" upper="${joint_upper_limit}" effort="${joint_effort}" velocity="${joint_velocity}"/>
         </joint>
         <transmission name="femur_transmission_${side}${position}">
             <type>transmission_interface/SimpleTransmission</type>
-            <joint name="femur_joint_${side}${position}">
+            <joint name="j_thigh_${side}${position}">
                 <hardwareInterface>EffortJointInterface</hardwareInterface>
             </joint>
@@ -135,9 +147,9 @@
             </actuator>
         </transmission>
-        <link name="femur_${side}${position}">
+        <link name="link_thigh_${side}${position}">
             <visual>
                 <origin xyz="0.0 0.0 0.0" rpy="0.0 0.0 0.0"/>
                 <geometry>
-                    <mesh filename="package://spider/meshes/femur_link.STL"/>
+                    <mesh filename="package://spider_description/meshes/xacro/femur_link.STL"/>
                 </geometry>
                 <material name="">
@@ -148,5 +160,5 @@
                 <origin xyz="0.0 0.0 0.0" rpy="0.0 0.0 0.0" />
                 <geometry>
-                    <mesh filename="package://spider/meshes/femur_link.STL"/>
+                    <mesh filename="package://spider_description/meshes/xacro/femur_link.STL"/>
                 </geometry>
                 <material name="">
@@ -155,23 +167,29 @@
             </collision>
             <inertial>
-                <origin xyz="0.0 0.0 0.0" rpy="0.0 0.0 0.0" />
-                <mass value="0.00001"/>
-                <inertia
-                    ixx="1.0" ixy="0.0"  ixz="0.0"
-                    iyy="1.0" iyz="0.0"
-                    izz="1.0" />
+            <origin
+                    xyz="0.040999769634667 -4.30568319366442E-08 0.000754475780533559"
+                    rpy="0 0 0" />
+                  <mass
+                    value="0.0953381260317791" />
+                  <inertia
+                    ixx="1.58226170549124E-05"
+                    ixy="7.18370173005665E-09"
+                    ixz="2.44292687080875E-07"
+                    iyy="9.74932250427542E-05"
+                    iyz="-1.77284495331422E-11"
+                    izz="9.24662892423645E-05" />
             </inertial>
         </link>
 <!-- tibia -->
-      <joint name="tibia_joint_${side}${position}" type="revolute">
+      <joint name="j_tibia_${side}${position}" type="revolute">
           <origin xyz="${femur_length} 0.0  0.0" rpy="${pi} 0.0 0.0"/>
-          <parent link="femur_${side}${position}"/>
-          <child link="tibia_${side}${position}"/>
-          <axis xyz="0.0 0.0 ${axis}"/>
+          <parent link="link_thigh_${side}${position}"/>
+          <child link="link_tibia_${side}${position}"/>
+          <axis xyz="0.0 0.0 ${axis_tibia}"/>
           <limit lower="${joint_lower_limit}" upper="${joint_upper_limit}" effort="${joint_effort}" velocity="${joint_velocity}"/>
       </joint>
       <transmission name="tibia_transmission_${side}${position}">
           <type>transmission_interface/SimpleTransmission</type>
-          <joint name="tibia_joint_${side}${position}">
+          <joint name="j_tibia_${side}${position}">
               <hardwareInterface>EffortJointInterface</hardwareInterface>
           </joint>
@@ -181,9 +199,9 @@
           </actuator>
       </transmission>
-      <link name="tibia_${side}${position}">
+      <link name="link_tibia_${side}${position}">
           <visual>
               <origin xyz="0.0 0.0 0.0" rpy="0.0 0.0 0.0"/>
               <geometry>
-                  <mesh filename="package://spider/meshes/tibia_link.STL"/>
+                  <mesh filename="package://spider_description/meshes/xacro/tibia_link.STL"/>
               </geometry>
               <material name="">
@@ -194,5 +212,5 @@
               <origin xyz="0.0 0.0 0.0" rpy="0.0 0.0 0.0" />
               <geometry>
-                  <mesh filename="package://spider/meshes/tibia_link.STL"/>
+                  <mesh filename="package://spider_description/meshes/xacro/tibia_link.STL"/>
               </geometry>
               <material name="">
@@ -201,10 +219,16 @@
           </collision>
           <inertial>
-              <origin xyz="0.0 0.0 0.0" rpy="0.0 0.0 0.0" />
-              <mass value="0.00001"/>
-              <inertia
-                  ixx="1.0" ixy="0.0"  ixz="0.0"
-                  iyy="1.0" iyz="0.0"
-                  izz="1.0" />
+          <origin
+                  xyz="0.0582130928710533 -4.8413205307532E-07 -0.000309754397326167"
+                  rpy="0 0 0" />
+                <mass
+                  value="0.0274685501932791" />
+                <inertia
+                  ixx="1.3790756851875E-05"
+                  ixy="1.86386884764665E-09"
+                  ixz="-2.70792447948708E-09"
+                  iyy="8.67578889959408E-05"
+                  iyz="1.52160816187718E-13"
+                  izz="7.87024641434495E-05" />
           </inertial>
       </link>
@@ -212,5 +236,5 @@
         <joint name="foot_joint_${side}${position}" type="fixed">
             <origin xyz="${tibia_length} 0.0 0.0" rpy="0.0 0.0 0.0" />
-            <parent link="tibia_${side}${position}" />
+            <parent link="link_tibia_${side}${position}" />
             <child link="foot_${side}${position}" />
         </joint>
@@ -218,18 +242,18 @@
             <inertial>
                 <origin xyz="0.0 0.0 0.0" rpy="0.0 0.0 0.0" />
-                <mass value="0.00001"/>
+                <mass value="0.00000001"/>
                 <inertia
-                    ixx="1.0" ixy="0.0"  ixz="0.0"
-                    iyy="1.0" iyz="0.0"
-                    izz="1.0" />
+                    ixx="0.01E-020" ixy="0.0"  ixz="0.0"
+                    iyy="0.01E-020" iyz="0.0"
+                    izz="0.01E-020" />
             </inertial>
         </link>
     </xacro:macro>
 <!-- Build robot model -->
-   <xacro:leg side="R" position="R" x="-0.170" y="-0.11" angle="-${pi*3/4}" axis="1"/>
-   <xacro:leg side="R" position="M" x="0.0" y="-0.132" angle="-${pi/2}" axis="1"/>
-   <xacro:leg side="R" position="F" x="0.170" y="-0.11" angle="-${pi/4}" axis="1"/>
-   <xacro:leg side="L" position="R" x="-0.170" y="0.11" angle="${pi*3/4}" axis="-1"/>
-   <xacro:leg side="L" position="M" x="0.0" y="0.132" angle="${pi/2}" axis="-1"/>
-   <xacro:leg side="L" position="F" x="0.170" y="0.11" angle="${pi/4}" axis="-1"/>
+<xacro:leg side="r" position="r" x="-0.170" y="-0.110" angle="-${pi*3/4}" axis_femur="1" axis_tibia="-1"/>
+<xacro:leg side="r" position="m" x="0.0" y="-0.1325" angle="-${pi/2}" axis_femur="1" axis_tibia="-1"/>
+<xacro:leg side="r" position="f" x="0.1778" y="-0.110" angle="-${pi/4}" axis_femur="1" axis_tibia="-1"/>
+<xacro:leg side="l" position="r" x="-0.170" y="0.110" angle="${pi*3/4}" axis_femur="-1" axis_tibia="1"/>
+<xacro:leg side="l" position="m" x="0.0" y="0.1325" angle="${pi/2}" axis_femur="-1" axis_tibia="1"/>
+<xacro:leg side="l" position="f" x="0.170" y="0.110" angle="${pi/4}" axis_femur="-1" axis_tibia="1"/>
 </robot>

File: spider_description/urdf/spider1.urdf (robot description, URDF)
Before this commit: robot spider_description, 19 links, 18 joints
Joints:
- joint j_c1_lf: axis 0 0 1 -> 0 0 -1
- joint j_c1_lm: axis 0 0 1 -> 0 0 -1
- joint j_c1_lr: axis 0 0 1 -> 0 0 -1
- joint j_c1_rf: axis 0 0 1 -> 0 0 -1
- joint j_c1_rm: axis 0 0 1 -> 0 0 -1
- joint j_c1_rr: axis 0 0 1 -> 0 0 -1
- joint j_thigh_lf: limit lower=-1.9199 upper=1.9199 effort=6.0 velocity=0.524 -> lower=-3.1416 upper=3.1416 effort=6.0 velocity=0.524
- joint j_thigh_lm: limit lower=-1.9199 upper=1.9199 effort=6.0 velocity=0.524 -> lower=-3.1416 upper=3.1416 effort=6.0 velocity=0.524
- joint j_thigh_lr: limit lower=-1.9199 upper=1.9199 effort=6.0 velocity=0.524 -> lower=-3.1416 upper=3.1416 effort=6.0 velocity=0.524
- joint j_thigh_rf: limit lower=-1.9199 upper=1.9199 effort=6.0 velocity=0.524 -> lower=-3.1416 upper=3.1416 effort=6.0 velocity=0.524
- joint j_thigh_rm: limit lower=-1.9199 upper=1.9199 effort=6.0 velocity=0.524 -> lower=-3.1416 upper=3.1416 effort=6.0 velocity=0.524
- joint j_thigh_rr: limit lower=-1.9199 upper=1.9199 effort=6.0 velocity=0.524 -> lower=-3.1416 upper=3.1416 effort=6.0 velocity=0.524
- joint j_tibia_lf: limit lower=-2.2689 upper=2.2689 effort=6.0 velocity=0.524 -> lower=-3.1416 upper=3.1416 effort=6.0 velocity=0.524
- joint j_tibia_lm: limit lower=-2.2689 upper=2.2689 effort=6.0 velocity=0.524 -> lower=-3.1416 upper=3.1416 effort=6.0 velocity=0.524
- joint j_tibia_lr: limit lower=-2.2689 upper=2.2689 effort=6.0 velocity=0.524 -> lower=-3.1416 upper=3.1416 effort=6.0 velocity=0.524
- joint j_tibia_rf: limit lower=-2.2689 upper=2.2689 effort=6.0 velocity=0.524 -> lower=-3.1416 upper=3.1416 effort=6.0 velocity=0.524
- joint j_tibia_rm: limit lower=-2.2689 upper=2.2689 effort=6.0 velocity=0.524 -> lower=-3.1416 upper=3.1416 effort=6.0 velocity=0.524
- joint j_tibia_rr: limit lower=-2.2689 upper=2.2689 effort=6.0 velocity=0.524 -> lower=-3.1416 upper=3.1416 effort=6.0 velocity=0.524
