Commit message: попытка выровнять походку 126263

File: spider_description/urdf/spider.xacro (robot description, xacro)
@@ -55,10 +55,10 @@
     </link>
     <!-- Joint properties -->
-   <xacro:property name="joint_lower_limit" value="-${3.14}"/>
-   <xacro:property name="joint_upper_limit" value="${3.14}"/>
+   <xacro:property name="joint_lower_limit" value="-2.00"/>
+   <xacro:property name="joint_upper_limit" value="2.00"/>
    <xacro:property name="joint_effort" value="6.0"/>
    <xacro:property name="joint_velocity" value="0.524"/>
     <!-- Leg macro -->
-    <xacro:macro name="leg" params="side position x y angle axis_femur axis_tibia">
+    <xacro:macro name="leg" params="side position x y angle axis_coxa axis_femur axis_tibia">
         <!-- leg position -->
         <joint name="leg_center_joint_${side}${position}" type="fixed">
@@ -82,5 +82,5 @@
            <parent link="leg_center_${side}${position}"/>
            <child link="link_c1_${side}${position}"/>
-           <axis xyz="0.0 0.0 1.0"/>
+           <axis xyz="0.0 0.0 ${axis_coxa}"/>
            <limit lower="${joint_lower_limit}" upper="${joint_upper_limit}" effort="${joint_effort}" velocity="${joint_velocity}"/>
        </joint>
@@ -268,9 +268,9 @@
       </gazebo>
 <!-- Build robot model -->
-<xacro:leg side="r" position="r" x="-0.170" y="-0.110" angle="-${pi*3/4}" axis_femur="1" axis_tibia="-1"/>
-<xacro:leg side="r" position="m" x="0.0" y="-0.1325" angle="-${pi/2}" axis_femur="1" axis_tibia="-1"/>
-<xacro:leg side="r" position="f" x="0.1778" y="-0.110" angle="-${pi/4}" axis_femur="1" axis_tibia="-1"/>
-<xacro:leg side="l" position="r" x="-0.170" y="0.110" angle="${pi*3/4}" axis_femur="-1" axis_tibia="1"/>
-<xacro:leg side="l" position="m" x="0.0" y="0.1325" angle="${pi/2}" axis_femur="-1" axis_tibia="1"/>
-<xacro:leg side="l" position="f" x="0.170" y="0.110" angle="${pi/4}" axis_femur="-1" axis_tibia="1"/>
+<xacro:leg side="r" position="r" x="-0.170" y="-0.110" angle="-${pi*3/4}" axis_femur="-1" axis_tibia="1" axis_coxa="1"/>
+<xacro:leg side="r" position="m" x="0.0" y="-0.1325" angle="-${pi/2}" axis_femur="-1" axis_tibia="1" axis_coxa="1"/>
+<xacro:leg side="r" position="f" x="0.1778" y="-0.110" angle="-${pi/4}" axis_femur="-1" axis_tibia="1" axis_coxa="1"/>
+<xacro:leg side="l" position="r" x="-0.170" y="0.110" angle="${pi*3/4}" axis_femur="1" axis_tibia="-1" axis_coxa="1"/>
+<xacro:leg side="l" position="m" x="0.0" y="0.1325" angle="${pi/2}" axis_femur="1" axis_tibia="-1" axis_coxa="1"/>
+<xacro:leg side="l" position="f" x="0.170" y="0.110" angle="${pi/4}" axis_femur="1" axis_tibia="-1" axis_coxa="1"/>
 </robot>

Commit message: начала делать движение ногами по команде

File: spider_description/urdf/spider.xacro (robot description, xacro)
@@ -18,5 +18,5 @@
         <parent link="base_link"/>
         <child link="body_link"/>
-        <origin xyz="0.0 0.0 0.064" rpy="0.0 0.0 0.0"/>
+        <origin xyz="0.0 0.0 0.0" rpy="0.0 0.0 0.0"/>
     </joint>
     <link name="body_link">
@@ -267,4 +267,21 @@
         </plugin>
       </gazebo>
+    <plugin name="p3d_base_controller" filename="libgazebo_ros_p3d.so">
+        <topicName>/aaaaaaaa</topicName>
+         <alwaysOn>true</alwaysOn>
+         <updateRate>50.0</updateRate>
+         <bodyName>body_link</bodyName>
+         <topicName>/ground_truth/state</topicName>
+         <gaussianNoise>0.01</gaussianNoise>
+         <frameName>world</frameName>
+         <xyzOffsets>0 0 0</xyzOffsets>
+         <rpyOffsets>0 0 0</rpyOffsets>
+       </plugin>
+<gazebo>
+    <plugin name="gazebo_ros_control" filename=" libgazebo_ros_p3d">
+      <!-- <robotNamespace></robotNamespace> -->
+      <topicName>/spider/odom_gazebo</topicName>
+    </plugin>
+  </gazebo>
 <!-- Build robot model -->
 <xacro:leg side="r" position="r" x="-0.170" y="-0.110" angle="-${pi*3/4}" axis_femur="-1" axis_tibia="1" axis_coxa="1"/>

Commit message: обновила алгоритм

File: spider_description/urdf/spider.xacro (robot description, xacro)
@@ -57,5 +57,5 @@
    <xacro:property name="joint_lower_limit" value="-2.00"/>
    <xacro:property name="joint_upper_limit" value="2.00"/>
-   <xacro:property name="joint_effort" value="6.0"/>
+   <xacro:property name="joint_effort" value="1.0"/>
    <xacro:property name="joint_velocity" value="0.524"/>
     <!-- Leg macro -->
